Commit message: Unify the URDF with Leo

File: panthera_description/urdf/panthera_ht_gripper.urdf (robot description, URDF)
Before this commit: robot Panthera-HT_description, 9 links, 8 joints
Links:
- removed link base_link
- added link panthera_base_link, mass 0.62922454; collision mesh filename=package://Panthera-HT_description/meshes/base_link.STL; visual mesh filename=package://Panthera-HT_description/meshes/base_link.STL
Joints:
- joint joint1: parent base_link -> panthera_base_link

File: panthera_description/urdf/panthera_ht_gripper.urdf.xacro (robot description, xacro)
@@ -3,5 +3,5 @@
      Commit Version: 1.6.0-4-g7f85cfe  Build Version: 1.6.7995.38578
      For more information, please see http://wiki.ros.org/sw_urdf_exporter -->
-<robot name="Panthera-HT_description" xmlns:xacro="http://www.ros.org/wiki/xacro">
+<robot name="leo" xmlns:xacro="http://www.ros.org/wiki/xacro">
   <!-- Xacro properties for commonly used values -->
   <xacro:property name="package_name" value="panthera_description" />
@@ -14,5 +14,5 @@
     <compiler meshdir="../meshes/" balanceinertia="true" discardvisual="false" />
   </mujoco>
-  <link name="base_link">
+  <link name="panthera_base_link">
     <inertial>
       <origin xyz="5.789e-05 -0.00015938 0.02298649" rpy="0 0 0" />
@@ -56,5 +56,5 @@
   <joint name="joint1" type="revolute">
     <origin xyz="0 0 0.0584" rpy="0 0 0" />
-    <parent link="base_link" />
+    <parent link="panthera_base_link" />
     <child link="link1" />
     <axis xyz="0 0 1" />

File: panthera_moveit/urdf/panthera_ht_moveit.urdf.xacro (robot description, xacro)
@@ -1,4 +1,4 @@
 <?xml version="1.0"?>
-<robot xmlns:xacro="http://www.ros.org/wiki/xacro" name="panthera_ht_description">
+<robot xmlns:xacro="http://www.ros.org/wiki/xacro" name="leo">
     <xacro:arg name="config_file" default="$(find panthera_moveit)/config/6dof_arm_params.yaml" />
     <xacro:arg name="control_mode" default="position_velocity" />
